File: elec/PCB_Ruler_V1_2024/Features.kicad_sch (KiCad schematic)
At the start: 0 parts

Commit message: IMU
Parts:
- added C1, C2, C3: 1uF, symbol Device:C
- added MT1: ICM-42670-P, IMU:XDCR_ICM-42670-P, symbol ICM-42670-P:ICM-42670-P
Connections:
- new net +3.3V: C1.1, C2.1, C3.1, MT1.5 (VDDIO), MT1.8 (VDD)
- new net GND: C1.2, C2.2, C3.2

Commit message: battery charger
Changed lines of the file:
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@@
+		)
+	)
+	(global_label "SDA"
+		(shape input)
+		(at 113.03 99.06 0)
+		(fields_autoplaced yes)
+		(effects
+			(font
+				(size 1.27 1.27)
+			)
+			(justify left)
+		)
+		(property "Intersheetrefs" "${INTERSHEET_REFS}"
+			(at 119.5833 99.06 0)
+			(effects
+				(font
+					(size 1.27 1.27)
+				)
+				(justify left)
+				(hide yes)
+			)
+		)
+	)
+	(global_label "SCL"
+		(shape input)
+		(at 113.03 101.6 0)
+		(fields_autoplaced yes)
+		(effects
+			(font
+				(size 1.27 1.27)
+			)
+			(justify left)
+		)
+		(property "Intersheetrefs" "${INTERSHEET_REFS}"
+			(at 119.5228 101.6 0)
+			(effects
+				(font
+					(size 1.27 1.27)
+				)
+				(justify left)
+				(hide yes)
+			)
 		)
 	)
@@
 		)
 		(instances
-			(project ""
+			(project "PCB_Ruler_V1_2024"
 				(path "/e39575e5-bba1-47dc-9ccf-32a84e6da237/ca7d0597-655a-4aee-bb72-0094cc7418df"
 					(reference "MT1")
@@
 		)
 		(instances
-			(project ""
+			(project "PCB_Ruler_V1_2024"
 				(path "/e39575e5-bba1-47dc-9ccf-32a84e6da237/ca7d0597-655a-4aee-bb72-0094cc7418df"
 					(reference "#PWR04")
@@
 		)
 		(instances
-			(project ""
+			(project "PCB_Ruler_V1_2024"
 				(path "/e39575e5-bba1-47dc-9ccf-32a84e6da237/ca7d0597-655a-4aee-bb72-0094cc7418df"
 					(reference "C1")
@@
 		)
 		(instances
-			(project ""
+			(project "PCB_Ruler_V1_2024"
 				(path "/e39575e5-bba1-47dc-9ccf-32a84e6da237/ca7d0597-655a-4aee-bb72-0094cc7418df"
 					(reference "#PWR02")

Commit message: this is for my strong girl
Parts:
- C1: value 1uF -> 0.1uF
- C2: value 1uF -> 2.2uF
- C3: value 1uF -> 10nF
Changed lines of the file:
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@@
 			)
 		)
-		(property "Value" "1uF"
+		(property "Value" "10nF"
 			(at 128.27 64.7699 0)
 			(effects
@@
 			)
 		)
-		(property "Value" "1uF"
+		(property "Value" "0.1uF"
 			(at 147.32 64.7699 0)
 			(effects
@@
 			)
 		)
-		(property "Value" "1uF"
+		(property "Value" "2.2uF"
 			(at 160.02 64.7699 0)
 			(effects

Commit message: Laser
Parts:
- added C7: 100nF, symbol Device:C
- added C8: 4.7 uF, symbol Device:C
- added R5, R6, R7: 10 k, symbol Device:R
- added U4: VL53L4CXV0DH/1, VL53L4CXV0DH/1:LGA12_STM, symbol VL53L4CXV0DH/1:VL53L4CXV0DH_1
Connections:
- net +3.3V: now also R5.1, R6.1, R7.1
- net GND: now also MT1.6 (GND), C7.2, C8.2, U4.12 (GND4), U4.2 (AVSSVCSEL), U4.3 (GND), U4.4 (GND2), U4.6 (GND3)
- net SCL: now also MT1.13 (AP_SCL/AP_SCLK), R6.2, U4.10 (SCL)
- net SDA: now also MT1.14 (AP_SDA/AP_SDIO/AP_SDI), R5.2, U4.9 (SDA)
- new net AVDD: C7.1, C8.1, U4.1 (AVDDVCSEL), U4.11 (AVDD)
- new net XSHUT: R7.2, U4.5 (XSHUT)
- no-connect marks 0 -> 1
Other:
- note added: "IMU"
- note added: "LASER"
- note added: "PULL UP RESISTORS"
- moved on the sheet: C1, C2, C3, MT1

Commit message: Almost finished schematic...
Parts:
- added C12: 1uF, symbol Device:C
- added U5: TCA9534PWR, TCA9534PWR:SOP65P640X120-16N, symbol TCA9534PWR:TCA9534PWR
Connections:
- net +3.3V: now also C12.1, U5.16 (VCC)
- net GND: now also C12.2, U5.1 (A0), U5.2 (A1), U5.3 (A2), U5.8 (GND)
- net SCL: now also U5.14 (SCL)
- net SDA: now also U5.15 (SDA)
- net XSHUT: now also U5.4 (P0)
- new net INT_IO_Extender: U5.13 (~{INT})
- new net IO2: U5.5 (P1)
- new net IO3: U5.6 (P2)
- new net IO4: U5.7 (P3)
- new net IO5: U5.9 (P4)
- new net IO6: U5.10 (P5)
- new net IO7: U5.11 (P6)
- new net IO8: U5.12 (P7)
- no-connect marks 1 -> 2
Other:
- note added: "IO EXTENDER"

Commit message: protection and Buttons
Connections:
- net IO2 renamed Button1
- net IO3 renamed Button2
- net IO4 renamed Button3
- net IO5 renamed Button4
- net IO6 renamed Button5

Commit message: started pcb
Parts:
- C10: renamed from C7; footprint (none) -> Capacitor_SMD:C_0603_1608Metric_Pad1.08x0.95mm_HandSolder
- C11: renamed from C8; footprint (none) -> Capacitor_SMD:C_0603_1608Metric_Pad1.08x0.95mm_HandSolder
- C12: footprint (none) -> Capacitor_SMD:C_0603_1608Metric_Pad1.08x0.95mm_HandSolder
- C7: renamed from C3; footprint (none) -> Capacitor_SMD:C_0603_1608Metric_Pad1.08x0.95mm_HandSolder
- C8: renamed from C1; footprint (none) -> Capacitor_SMD:C_0603_1608Metric_Pad1.08x0.95mm_HandSolder
- C9: renamed from C2; footprint (none) -> Capacitor_SMD:C_0603_1608Metric_Pad1.08x0.95mm_HandSolder
- R10: renamed from R5; footprint (none) -> Resistor_SMD:R_0603_1608Metric_Pad0.98x0.95mm_HandSolder
- R11: renamed from R6; footprint (none) -> Resistor_SMD:R_0603_1608Metric_Pad0.98x0.95mm_HandSolder
- R9: renamed from R7; footprint (none) -> Resistor_SMD:R_0603_1608Metric_Pad0.98x0.95mm_HandSolder
- renumbered U5 to U4, U4 to U5
