File: elec/PCB_Ruler_V1_2024/PCB_Ruler_V1_2024.kicad_pcb (KiCad board)
At the start: 2 copper layers, 51 parts, among them J1 USB-C, J2 S2B-XH-A-1LFSN, SW1 CS1213AGF260, SW2 CS1213AGF260, SW3 CS1213AGF260, SW4 CS1213AGF260, SW5 CS1213AGF260, SW6 CS1213AGF260, SW7 CS1213AGF260, U1 ESP32-C3-WROOM-02-H4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

Commit message: idk
Parts:
- moved D2 57.6 mm to (219.8, 130.7)
- moved U5 57.6 mm to (182.0, 133.2)
- moved C13 57.6 mm to (147.9, 135.8)
- moved C6 57.6 mm to (210.2, 143.4)
- moved D1 57.6 mm to (219.8, 132.6)
- moved S1 57.6 mm to (214.8, 126.8)
- moved SW2 57.6 mm to (224.5, 126.9)
- moved SW5 57.6 mm to (150.8, 135.8)
- moved U3 57.6 mm to (210.4, 136.6)
- moved C5 57.6 mm to (210.2, 140.9)
- moved J1 57.6 mm to (222.0, 142.9)
- moved J3 57.6 mm to (143.1, 135.4)
- moved R12 57.6 mm to (150.9, 130.9)
- moved R13 57.6 mm to (160.6, 131.1)
- moved R14 57.6 mm to (150.6, 140.9)
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Other:
- board outline added: 155 x 30 mm

Commit message: Je les ai mis ensemble mais pour les places en tant que tel pas sur , pas sur
Parts:
- moved C1 166.8 mm to (216.0, 146.0)
- moved C2 166.5 mm to (216.0, 148.0)
- moved R4 158.7 mm to (216.0, 143.0)
- moved R3 158.4 mm to (216.0, 140.0)
- moved R2 158.2 mm to (216.0, 137.0)
- moved R1 158.0 mm to (216.0, 134.0)
- moved C8 144.5 mm to (198.0, 144.0)
- moved C9 144.5 mm to (198.0, 146.5)
- moved C7 144.2 mm to (198.0, 141.0)
- moved R10 136.5 mm to (202.6, 138.0)
- moved R9 136.5 mm to (202.6, 135.5)
- moved R11 136.5 mm to (202.6, 140.5)
- moved MT1 129.9 mm to (198.0, 137.5)
- moved C12 125.9 mm to (190.5, 132.5)
- moved C10 124.3 mm to (179.0, 140.5), turned to 180 degrees
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
Commit message: yeah
Parts:
- moved C5 11.2 mm to (197.5, 126.5), turned to 180 degrees
- moved J1 8.73 mm to (222.5, 148.5), turned to 0 degrees
- moved C6 6.71 mm to (206.5, 126.5), turned to 0 degrees
- moved J2 2.11 mm to (112.2, 134.7)
- moved C1 1.86 mm to (214.1, 146.0)
- moved C2 1.86 mm to (214.1, 148.0)
- moved R1 1.86 mm to (214.1, 134.0)
- moved R2 1.86 mm to (214.1, 137.0)
- moved R3 1.86 mm to (214.1, 140.0)
- moved R4 1.86 mm to (214.1, 143.0)
- moved U3 1.50 mm to (202.0, 127.5), turned to 0 degrees
- moved S1 0.66 mm to (214.8, 127.5)

Commit message: modifs :D
Parts:
- moved D3 97.0 mm to (220.0, 135.0), turned to 180 degrees
- moved R5 84.9 mm to (213.2, 135.2)
- moved R6 84.9 mm to (213.3, 138.2)
- moved U2 84.9 mm to (208.0, 136.5)
- moved C3 75.2 mm to (208.1, 143.0)
- moved C4 74.3 mm to (208.0, 140.5)
- moved C1 34.9 mm to (244.0, 128.0)
- moved J2 32.1 mm to (142.2, 146.2), turned to 90 degrees
- moved R2 26.9 mm to (239.5, 128.0)
- moved R9 25.0 mm to (178.8, 143.0), turned to 90 degrees
- moved R1 18.9 mm to (232.1, 128.0)
- moved R4 13.1 mm to (225.5, 136.5)
- moved R3 11.4 mm to (225.5, 140.0)
- moved C2 10.1 mm to (219.6, 139.5)
- moved C12 9.07 mm to (182.4, 128.5), turned to 180 degrees
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
Commit message: allo
Parts:
- moved R7 71.1 mm to (204.1, 136.0)
- moved R8 71.0 mm to (204.1, 133.5)
- moved D3 64.8 mm to (155.5, 128.5)
- moved S1 19.4 mm to (196.0, 132.5), turned to 180 degrees
- moved R5 12.1 mm to (209.0, 146.5), turned to 90 degrees
- moved R10 11.1 mm to (191.0, 141.1)
- moved R11 11.1 mm to (191.0, 143.6)
- moved D1 9.92 mm to (226.5, 140.0)
- moved D2 9.92 mm to (226.5, 138.1)
- moved C6 8.64 mm to (214.6, 129.4)
- moved U3 8.53 mm to (210.0, 130.4)
- moved C5 8.17 mm to (205.1, 129.4)
- moved C10 7.89 mm to (179.7, 139.6), turned to 90 degrees
- moved C7 7.19 mm to (195.5, 145.6)
- moved MT1 7.19 mm to (195.5, 142.1)
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
Commit message: started the pcb
Parts:
- moved D3 50.9 mm to (204.2, 143.6), turned to 0 degrees
- moved C2 28.6 mm to (243.0, 126.6), turned to 90 degrees
- moved D2 7.01 mm to (225.6, 145.0)
- moved D1 5.22 mm to (228.0, 145.0), turned to 0 degrees
- moved C1 4.98 mm to (239.2, 126.5), turned to 90 degrees
- moved J1 3.54 mm to (219.0, 148.5)
- moved R2 3.13 mm to (236.8, 126.5), turned to 90 degrees
- moved C6 2.86 mm to (217.5, 129.5)
- moved R1 1.55 mm to (232.4, 126.5), turned to 90 degrees
- moved C5 1.14 mm to (204.0, 129.4)
- moved R18 0.25 mm to (150.0, 138.4)
- moved R12 0.25 mm to (160.0, 132.8)
- moved R13 0.25 mm to (171.0, 132.8)
- moved R14 0.25 mm to (160.0, 141.8)
- moved R16 0.25 mm to (171.0, 141.8)
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Connections:
- C12 pad 1: +3.3V -> AVDD
- C13 pad 1: +3.3V -> AVDD
- C2 pad 1: +3.3V -> AVDD
- C6 pad 1: +3V3 -> AVDD
- C7 pad 1: +3.3V -> AVDD
- C8 pad 1: +3.3V -> AVDD
- C9 pad 1: +3.3V -> AVDD
- J3 pad 10: +3.3V -> AVDD
- MT1 pad 1: unconnected-(MT1-AP_SDO/AP_AD0-Pad1) -> AVDD
- MT1 pad 12: unconnected-(MT1-AP_CS-Pad12) -> AVDD
- MT1 pad 4: unconnected-(MT1-INT1/INT-Pad4) -> INT1_IMU
- MT1 pad 5: +3.3V -> AVDD
- MT1 pad 7: unconnected-(MT1-FSYNC-Pad7) -> GND
- MT1 pad 8: +3.3V -> AVDD
- MT1 pad 9: unconnected-(MT1-INT2-Pad9) -> INT2_IMU
- R1 pad 2: +3.3V -> AVDD
- R10 pad 1: +3.3V -> AVDD
- R11 pad 1: +3.3V -> AVDD
- R12 pad 1: +3.3V -> AVDD
- R13 pad 1: +3.3V -> AVDD
- R14 pad 1: +3.3V -> AVDD
- R15 pad 1: +3.3V -> CS_Ecran
- R15 pad 2: CS_Ecran -> GND
- R16 pad 1: +3.3V -> AVDD
- R17 pad 1: +3.3V -> AVDD
- R18 pad 1: +3.3V -> AVDD
- R2 pad 2: +3.3V -> AVDD
- R9 pad 1: +3.3V -> AVDD
- U1 pad 1: +3.3V -> AVDD
- U3 pad 5: +3V3 -> AVDD
- U4 pad 16: +3.3V -> AVDD
Routing:
- net AVDD: track 0.00 -> 241.0 mm
- net Vbat+: track 0.00 -> 84.6 mm, vias 0 -> 3
- net USB_D+: track 0.00 -> 29.3 mm
- net Vin: track 0.00 -> 28.5 mm
- net USB_D-: track 0.00 -> 28.4 mm
- net +5V: track 0.00 -> 27.1 mm, vias 0 -> 2
- net Net-(J1-CC1): track 0.00 -> 9.36 mm
- net Net-(D3-K): track 0.00 -> 7.32 mm
- net Net-(J1-CC2): track 0.00 -> 5.53 mm, vias 0 -> 2
- net Net-(J3-LEDA): track 0.00 -> 4.87 mm
- net Net-(U2-STAT): track 0.00 -> 2.26 mm
- net Net-(U2-PROG): track 0.00 -> 2.26 mm

Commit message: meeting miriam
Parts:
- moved C5 0.86 mm to (204.1, 128.6), turned to 90 degrees
Routing:
- net AVDD: track 241.0 -> 243.3 mm
- net +5V: track 27.1 -> 25.2 mm

Commit message: Hi handsome :)
Parts:
- moved R10 1.00 mm to (190.0, 141.1)
- moved R11 1.00 mm to (190.0, 143.6)
Routing:
- net Touch0: track 0.00 -> 142.2 mm, vias 0 -> 2
- net Touch1: track 0.00 -> 138.6 mm, vias 0 -> 2
- net SPI_MOSI: track 0.00 -> 115.2 mm, vias 0 -> 2
- net SPI_CLK: track 0.00 -> 110.7 mm, vias 0 -> 2
- net RESET_Ecran: track 0.00 -> 106.9 mm, vias 0 -> 2
- net RS: track 0.00 -> 106.5 mm, vias 0 -> 2
- net CS_Ecran: track 0.00 -> 99.8 mm, vias 0 -> 2
- net SCL: track 0.00 -> 50.2 mm, vias 0 -> 4
- net SDA: track 0.00 -> 31.2 mm
- net XSHUT: track 0.00 -> 22.7 mm, vias 0 -> 2
- net AVDD: track 243.3 -> 249.5 mm
- net GND: track 0.00 -> 2.81 mm
