File: elec/PCB_Ruler_V1_2024/MCU_ESP32-C3.kicad_sch (KiCad schematic)
At the start: 13 parts, among them J1 USB-C, J4 61300211121, SW1 CS1213AGF260, SW2 CS1213AGF260, U1 ESP32-C3-WROOM-02-H4

Commit message: coucou v2
Other:
- company: (none) -> FRANK_LAU
- title: (none) -> MCU_RULER 2024
- moved on the sheet: C2
Changed lines of the file:
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@@
 	(generator_version "8.0")
 	(paper "A4")
+	(title_block
+		(title "MCU_RULER 2024")
+		(date "2024-12-27")
+		(rev "A")
+		(company "FRANK_LAU")
+	)
 	(junction
 		(at 157.48 116.84)
@@
 	(wire
 		(pts
-			(xy 36.83 168.91) (xy 36.83 171.45)
+			(xy 53.34 133.35) (xy 53.34 135.89)
 		)
 		(stroke
@@
 	(wire
 		(pts
-			(xy 36.83 179.07) (xy 36.83 181.61)
+			(xy 53.34 143.51) (xy 53.34 146.05)
 		)
 		(stroke
@@
 	(symbol
 		(lib_id "power:GND")
-		(at 36.83 181.61 0)
+		(at 53.34 146.05 0)
 		(unit 1)
 		(exclude_from_sim no)
@@
 		(fields_autoplaced yes)
 		(property "Reference" "#PWR016"
-			(at 36.83 187.96 0)
+			(at 53.34 152.4 0)
 			(effects
 				(font
@@
 		)
 		(property "Value" "GND"
-			(at 36.83 186.69 0)
+			(at 53.34 151.13 0)
 			(effects
 				(font
@@
 		)
 		(property "Footprint" ""
-			(at 36.83 181.61 0)
+			(at 53.34 146.05 0)
 			(effects
 				(font
@@
 		)
 		(property "Datasheet" ""
-			(at 36.83 181.61 0)
+			(at 53.34 146.05 0)
 			(effects
 				(font
@@
 		)
 		(property "Description" "Power symbol creates a global label with name \"GND\" , ground"
-			(at 36.83 181.61 0)
+			(at 53.34 146.05 0)
 			(effects
 				(font
@@
 	(symbol
 		(lib_id "power:+3.3V")
-		(at 36.83 168.91 0)
+		(at 53.34 133.35 0)
 		(unit 1)
 		(exclude_from_sim no)
@@
 		(fields_autoplaced yes)
 		(property "Reference" "#PWR015"
-			(at 36.83 172.72 0)
+			(at 53.34 137.16 0)
 			(effects
 				(font
@@
 		)
 		(property "Value" "+3.3V"
-			(at 36.83 163.83 0)
+			(at 53.34 128.27 0)
 			(effects
 				(font
@@
 		)
 		(property "Footprint" ""
-			(at 36.83 168.91 0)
+			(at 53.34 133.35 0)
 			(effects
 				(font
@@
 		)
 		(property "Datasheet" ""
-			(at 36.83 168.91 0)
+			(at 53.34 133.35 0)
 			(effects
 				(font
@@
 		)
 		(property "Description" "Power symbol creates a global label with name \"+3.3V\""
-			(at 36.83 168.91 0)
+			(at 53.34 133.35 0)
 			(effects
 				(font
@@
 	(symbol
 		(lib_id "Device:C")
-		(at 36.83 175.26 0)
+		(at 53.34 139.7 0)
 		(unit 1)
 		(exclude_from_sim no)
@@
 		(fields_autoplaced yes)
 		(property "Reference" "C2"
-			(at 40.64 173.9899 0)
+			(at 57.15 138.4299 0)
 			(effects
 				(font
@@
 		)
 		(property "Value" "1uF"
-			(at 40.64 176.5299 0)
+			(at 57.15 140.9699 0)
 			(effects
 				(font
@@
 		)
 		(property "Footprint" "Capacitor_SMD:C_0603_1608Metric_Pad1.08x0.95mm_HandSolder"
-			(at 37.7952 179.07 0)
+			(at 54.3052 143.51 0)
 			(effects
 				(font
@@
 		)
 		(property "Datasheet" "~"
-			(at 36.83 175.26 0)
+			(at 53.34 139.7 0)
 			(effects
 				(font
@@
 		)
 		(property "Description" "Unpolarized capacitor"
-			(at 36.83 175.26 0)
+			(at 53.34 139.7 0)
 			(effects
 				(font
