File: elec/PCB_Ruler_V1_2024/Screen.kicad_sch (KiCad schematic)
At the start: 0 parts

Commit message: battery charger
Parts:
- added J1: ~, Connector_FFC-FPC:Hirose_FH12-13S-0.5SH_1x13-1MP_P0.50mm_Horizontal, symbol ConnectorScreen:Header1x13
- added R1: 20 - 25 ohm, symbol Device:R
Connections:
- new net: J1.12 (LEDA), R1.2
- new net +3.3V: J1.10 (VDD)
- new net CS_Ecran: J1.7 (CS)
- new net GND: J1.11 (LEDK), J1.13 (GND), J1.8 (GND)
- new net RESET_Ecran: J1.6 (RESET)
- new net RS: J1.5 (RS)
- new net SPI_CLK: J1.4 (SCL)
- new net SPI_MOSI: J1.3 (SDA)
- new net Touch0: J1.1 (TP0)
- new net Touch1: J1.2 (TP1)
- no-connect marks 0 -> 1

Commit message: Almost finished schematic...
Parts:
- added C11: 1uF, symbol Device:C
- added R8: 10 k, symbol Device:R
- added SW3, SW4, SW5, SW6, SW7: CS1213AGF260, CS1213AGF260:SW_CS1213AGF260_CRS, symbol CS1213AGF260:CS1213AGF260
Connections:
- net +3.3V: now also R1.1, C11.1, R8.1
- net CS_Ecran: now also R8.2
- net GND: now also C11.2
Other:
- note added: "Connecteur Ecran"
- note added: "PULL-UP"
- moved on the sheet: J1, R1

Commit message: protection and Buttons
Parts:
- added R11, R13, R14, R15, R16: 10 k, symbol Device:R
Connections:
- net +3.3V: now also R11.1, R13.1, R14.1, R15.1, R16.1
- net GND: now also SW3.2, SW4.2, SW5.2, SW6.2, SW7.2
- net Button3: now reaches SW5.1
- net Button3: now also R14.2
- net Button2: now reaches SW4.1
- net Button2: now also R13.2
- net Button4: now reaches SW6.1
- net Button4: now also R15.2
- net Button1: now reaches SW3.1
- net Button1: now also R11.2
- net Button5: now reaches SW7.1
- net Button5: now also R16.2
Other:
- note added: "NAVIGATIONEL BUTTON"
- moved on the sheet: SW3, SW4, SW5, SW6, SW7

Commit message: started pcb
Parts:
- removed R11, R15: 10 k, symbol Device:R
- added R12, R17: 10 k, Resistor_SMD:R_0603_1608Metric_Pad0.98x0.95mm_HandSolder, symbol Device:R
- C13: renamed from C11; footprint (none) -> Capacitor_SMD:C_0603_1608Metric_Pad1.08x0.95mm_HandSolder
- R13, R14, R16: footprint (none) -> Resistor_SMD:R_0603_1608Metric_Pad0.98x0.95mm_HandSolder
- R15: renamed from R8; footprint (none) -> Resistor_SMD:R_0603_1608Metric_Pad0.98x0.95mm_HandSolder
- R18: renamed from R1; footprint (none) -> Resistor_SMD:R_0603_1608Metric_Pad0.98x0.95mm_HandSolder
- renumbered J1 to J3
Connections:
- net +3.3V: now also R12.1, R17.1
- net Button1: now also R12.2
- net Button4: now also R16.2
- net Button5: now also R17.2; no longer R16.2

Commit message: pull down
Connections:
- net +3.3V: no longer R15.1
- net CS_Ecran: now also R15.1; no longer R15.2
- net GND: now also R15.2
Other:
- note added: "PULL-DOWN"
- note removed: "PULL-UP"
- moved on the sheet: R15
Changed lines of the file:
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@@
-	(wire
-		(pts
-			(xy 250.19 44.45) (xy 250.19 43.18)
-		)
-		(stroke
-			(width 0)
-			(type default)
-		)
-	)
 	(wire
 		(pts
@@
 	(wire
 		(pts
-			(xy 250.19 33.02) (xy 250.19 35.56)
-		)
-		(stroke
-			(width 0)
-			(type default)
-		)
-	)
-	(wire
-		(pts
 			(xy 142.24 43.18) (xy 142.24 44.45)
 		)
@@
 	(wire
 		(pts
-			(xy 250.19 44.45) (xy 248.92 44.45)
-		)
-		(stroke
-			(width 0)
-			(type default)
-		)
-	)
-	(wire
-		(pts
 			(xy 237.49 101.6) (xy 237.49 109.22)
 		)
@@
 	(wire
 		(pts
+			(xy 250.19 29.21) (xy 250.19 30.48)
+		)
+		(stroke
+			(width 0)
+			(type default)
+		)
+	)
+	(wire
+		(pts
 			(xy 123.19 40.64) (xy 123.19 43.18)
 		)
@@
 	(wire
 		(pts
+			(xy 248.92 29.21) (xy 250.19 29.21)
+		)
+		(stroke
+			(width 0)
+			(type default)
+		)
+	)
+	(wire
+		(pts
 			(xy 77.47 40.64) (xy 77.47 43.18)
 		)
@@
 		(pts
 			(xy 232.41 111.76) (xy 240.03 111.76)
+		)
+		(stroke
+			(width 0)
+			(type default)
+		)
+	)
+	(wire
+		(pts
+			(xy 250.19 38.1) (xy 250.19 39.37)
 		)
 		(stroke
@@
 		)
 	)
-	(text "PULL-UP"
+	(text "PULL-DOWN"
 		(exclude_from_sim no)
 		(at 247.396 19.812 0)
@@
 		)
 	)
-	(global_label "CS_Ecran"
+	(global_label "Button5"
 		(shape input)
-		(at 248.92 44.45 180)
+		(at 101.6 72.39 180)
 		(fields_autoplaced yes)
 		(effects
@@
 		)
 		(property "Intersheetrefs" "${INTERSHEET_REFS}"
-			(at 237.1659 44.45 0)
+			(at 91.2369 72.39 0)
 			(effects
 				(font
@@
 		)
 	)
-	(global_label "Button5"
+	(global_label "Button3"
 		(shape input)
-		(at 101.6 72.39 180)
+		(at 120.65 43.18 180)
 		(fields_autoplaced yes)
 		(effects
@@
 		)
 		(property "Intersheetrefs" "${INTERSHEET_REFS}"
-			(at 91.2369 72.39 0)
+			(at 110.2869 43.18 0)
 			(effects
 				(font
@@
 		)
 	)
-	(global_label "Button3"
+	(global_label "RESET_Ecran"
 		(shape input)
-		(at 120.65 43.18 180)
+		(at 234.95 96.52 180)
 		(fields_autoplaced yes)
 		(effects
@@
 		)
 		(property "Intersheetrefs" "${INTERSHEET_REFS}"
-			(at 110.2869 43.18 0)
+			(at 219.9303 96.52 0)
 			(effects
 				(font
@@
 		)
 	)
-	(global_label "RESET_Ecran"
+	(global_label "Touch1"
 		(shape input)
-		(at 234.95 96.52 180)
+		(at 234.95 86.36 180)
 		(fields_autoplaced yes)
 		(effects
@@
 		)
 		(property "Intersheetrefs" "${INTERSHEET_REFS}"
-			(at 219.9303 96.52 0)
+			(at 225.2521 86.36 0)
 			(effects
 				(font
@@
 		)
 	)
-	(global_label "Touch1"
+	(global_label "CS_Ecran"
 		(shape input)
-		(at 234.95 86.36 180)
+		(at 234.95 99.06 180)
 		(fields_autoplaced yes)
 		(effects
@@
 		)
 		(property "Intersheetrefs" "${INTERSHEET_REFS}"
-			(at 225.2521 86.36 0)
+			(at 223.1959 99.06 0)
 			(effects
 				(font
@@
 	(global_label "CS_Ecran"
 		(shape input)
-		(at 234.95 99.06 180)
+		(at 248.92 29.21 180)
 		(fields_autoplaced yes)
 		(effects
@@
 		)
 		(property "Intersheetrefs" "${INTERSHEET_REFS}"
-			(at 223.1959 99.06 0)
+			(at 237.1659 29.21 0)
 			(effects
 				(font
@@
 	)
 	(symbol
+		(lib_id "power:GND")
+		(at 250.19 39.37 0)
+		(unit 1)
+		(exclude_from_sim no)
+		(in_bom yes)
+		(on_board yes)
+		(dnp no)
+		(fields_autoplaced yes)
+		(property "Reference" "#PWR046"
+			(at 250.19 45.72 0)
+			(effects
+				(font
+					(size 1.27 1.27)
+				)
+				(hide yes)
+			)
+		)
+		(property "Value" "GND"
+			(at 250.19 44.45 0)
+			(effects
+				(font
+					(size 1.27 1.27)
+				)
+			)
+		)
+		(property "Footprint" ""
+			(at 250.19 39.37 0)
+			(effects
+				(font
+					(size 1.27 1.27)
+				)
+				(hide yes)
+			)
+		)
+		(property "Datasheet" ""
+			(at 250.19 39.37 0)
+			(effects
+				(font
+					(size 1.27 1.27)
+				)
+				(hide yes)
+			)
+		)
+		(property "Description" "Power symbol creates a global label with name \"GND\" , ground"
+			(at 250.19 39.37 0)
+			(effects
+				(font
+					(size 1.27 1.27)
+				)
+				(hide yes)
+			)
+		)
+		(pin "1"
+		)
+		(instances
+			(project "PCB_Ruler_V1_2024"
+				(path "/e39575e5-bba1-47dc-9ccf-32a84e6da237/aecab3f5-8510-42f3-bc78-9784f4de281a"
+					(reference "#PWR046")
+					(unit 1)
+				)
+			)
+		)
+	)
+	(symbol
 		(lib_id "ConnectorScreen:Header1x13")
 		(at 242.57 78.74 0)
@@
 	(symbol
 		(lib_id "Device:R")
-		(at 250.19 39.37 0)
+		(at 250.19 34.29 0)
 		(unit 1)
 		(exclude_from_sim no)
@@
 		(fields_autoplaced yes)
 		(property "Reference" "R15"
-			(at 252.73 38.0999 0)
+			(at 252.73 33.0199 0)
 			(effects
 				(font
@@
 		)
 		(property "Value" "10 k"
-			(at 252.73 40.6399 0)
+			(at 252.73 35.5599 0)
 			(effects
 				(font
@@
 		)
 		(property "Footprint" "Resistor_SMD:R_0603_1608Metric_Pad0.98x0.95mm_HandSolder"
-			(at 248.412 39.37 90)
+			(at 248.412 34.29 90)
 			(effects
 				(font
@@
 		)
 		(property "Datasheet" "~"
-			(at 250.19 39.37 0)
+			(at 250.19 34.29 0)
 			(effects
 				(font
@@
 		)
 		(property "Description" "Resistor"
-			(at 250.19 39.37 0)
+			(at 250.19 34.29 0)
 			(effects
 				(font
@@
 					(unit 1)
 				)
-			)
-		)
-	)
-	(symbol
-		(lib_id "power:+3.3V")
-		(at 250.19 33.02 0)
-		(unit 1)
-		(exclude_from_sim no)
-		(in_bom yes)
-		(on_board yes)
-		(dnp no)
-		(fields_autoplaced yes)
-		(property "Reference" "#PWR046"
-			(at 250.19 36.83 0)
-			(effects
-				(font
-					(size 1.27 1.27)
-				)
-				(hide yes)
-			)
-		)
-		(property "Value" "+3.3V"
-			(at 250.19 27.94 0)
-			(effects
-				(font
-					(size 1.27 1.27)
-				)
-			)
-		)
-		(property "Footprint" ""
-			(at 250.19 33.02 0)
-			(effects
-				(font
-					(size 1.27 1.27)
-				)
-				(hide yes)
-			)
-		)
-		(property "Datasheet" ""
-			(at 250.19 33.02 0)
-			(effects
-				(font
-					(size 1.27 1.27)
-				)
-				(hide yes)
-			)
-		)
-		(property "Description" "Power symbol creates a global label with name \"+3.3V\""
-			(at 250.19 33.02 0)
-			(effects
-				(font
-					(size 1.27 1.27)
-				)
-				(hide yes)
-			)
-		)
-		(pin "1"
-		)
-		(instances
-			(project "PCB_Ruler_V1_2024"
-				(path "/e39575e5-bba1-47dc-9ccf-32a84e6da237/aecab3f5-8510-42f3-bc78-9784f4de281a"
-					(reference "#PWR046")
-					(unit 1)
-				)

Commit message: coucou v2
Other:
- title: (none) -> ÉCRAN_RULER 2024
- moved on the sheet: C13
Changed lines of the file:
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@@
 	(generator_version "8.0")
 	(paper "A4")
+	(title_block
+		(title "ÉCRAN_RULER 2024")
+		(date "2024-12-27")
+		(rev "A")
+	)
 	(junction
 		(at 123.19 43.18)
@@
 	(wire
 		(pts
-			(xy 25.4 181.61) (xy 25.4 184.15)
+			(xy 57.15 128.27) (xy 57.15 130.81)
 		)
 		(stroke
@@
 	(wire
 		(pts
-			(xy 25.4 171.45) (xy 25.4 173.99)
+			(xy 57.15 118.11) (xy 57.15 120.65)
 		)
 		(stroke
@@
 	(symbol
 		(lib_id "Device:C")
-		(at 25.4 177.8 0)
+		(at 57.15 124.46 0)
 		(unit 1)
 		(exclude_from_sim no)
@@
 		(fields_autoplaced yes)
 		(property "Reference" "C13"
-			(at 29.21 176.5299 0)
+			(at 60.96 123.1899 0)
 			(effects
 				(font
@@
 		)
 		(property "Value" "1uF"
-			(at 29.21 179.0699 0)
+			(at 60.96 125.7299 0)
 			(effects
 				(font
@@
 		)
 		(property "Footprint" "Capacitor_SMD:C_0603_1608Metric_Pad1.08x0.95mm_HandSolder"
-			(at 26.3652 181.61 0)
+			(at 58.1152 128.27 0)
 			(effects
 				(font
@@
 		)
 		(property "Datasheet" "~"
-			(at 25.4 177.8 0)
+			(at 57.15 124.46 0)
 			(effects
 				(font
@@
 		)
 		(property "Description" "Unpolarized capacitor"
-			(at 25.4 177.8 0)
+			(at 57.15 124.46 0)
 			(effects
 				(font
@@
 	(symbol
 		(lib_id "power:GND")
-		(at 25.4 184.15 0)
+		(at 57.15 130.81 0)
 		(unit 1)
 		(exclude_from_sim no)
@@
 		(fields_autoplaced yes)
 		(property "Reference" "#PWR057"
-			(at 25.4 190.5 0)
+			(at 57.15 137.16 0)
 			(effects
 				(font
@@
 		)
 		(property "Value" "GND"
-			(at 25.4 189.23 0)
+			(at 57.15 135.89 0)
 			(effects
 				(font
@@
 		)
 		(property "Footprint" ""
-			(at 25.4 184.15 0)
+			(at 57.15 130.81 0)
 			(effects
 				(font
@@
 		)
 		(property "Datasheet" ""
-			(at 25.4 184.15 0)
+			(at 57.15 130.81 0)
 			(effects
 				(font
@@
 		)
 		(property "Description" "Power symbol creates a global label with name \"GND\" , ground"
-			(at 25.4 184.15 0)
+			(at 57.15 130.81 0)
 			(effects
 				(font
@@
 	(symbol
 		(lib_id "power:+3.3V")
-		(at 25.4 171.45 0)
+		(at 57.15 118.11 0)
 		(unit 1)
 		(exclude_from_sim no)
@@
 		(fields_autoplaced yes)
 		(property "Reference" "#PWR056"
-			(at 25.4 175.26 0)
+			(at 57.15 121.92 0)
 			(effects
 				(font
@@
 		)
 		(property "Value" "+3.3V"
-			(at 25.4 166.37 0)
+			(at 57.15 113.03 0)
 			(effects
 				(font
@@
 		)
 		(property "Footprint" ""
-			(at 25.4 171.45 0)
+			(at 57.15 118.11 0)
 			(effects
 				(font
@@
 		)
 		(property "Datasheet" ""
-			(at 25.4 171.45 0)
+			(at 57.15 118.11 0)
 			(effects
 				(font
@@
 		)
 		(property "Description" "Power symbol creates a global label with name \"+3.3V\""
-			(at 25.4 171.45 0)
-			(effects
-				(font
+			(at 57.15 118.11 0)
+			(effects
+				(font
